File: ftdi.kicad_sch (KiCad schematic)
At the start: 31 parts, among them J1 USB4105-GF-A, U10 TPD4E02B04DQA, U11 TAR5S33UTE85LF, U2 FT4232H-56Q, Y1 ABM8G-12.000MHZ-18-D2Y-T

Commit message: Loclib
Parts:
- C8: footprint antmicro-footprints:0603-cap -> arty-mpw-tester-footprints:0603-cap; symbol antmicroCapacitors0603:C_10u_0603 -> arty-mpw-tester:C_10u_0603
- FB1, FB2, FB3: footprint antmicro-footprints:0603-res -> arty-mpw-tester-footprints:0603-res; symbol antmicroFerriteBeadsandChips:BLM18SG121TN1D -> arty-mpw-tester:BLM18SG121TN1D
- U11: footprint antmicro-footprints:SOT-353 -> arty-mpw-tester-footprints:SOT-353; symbol antmicroPMICVoltageRegulatorsLinear:TAR5S33UTE85LF -> arty-mpw-tester:TAR5S33UTE85LF
- U2: footprint antmicro-footprints:QFN-56-1EP_8x8mm_P0.5mm_EP5.5.9x5.9mm -> arty-mpw-tester-footprints:QFN-56-1EP_8x8mm_P0.5mm_EP5.5.9x5.9mm; symbol antmicroInterfaceControllers:FT4232H-56Q -> arty-mpw-tester:FT4232H-56Q
Changed lines of the file:
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@@
     (pin "2")
   )
-  (symbol (lib_id "antmicroInterfaceControllers:FT4232H-56Q") (at 124.46 167.64 0) (unit 1)
+  (symbol (lib_id "arty-mpw-tester:FT4232H-56Q") (at 124.46 167.64 0) (unit 1)
     (in_bom yes) (on_board yes) (fields_autoplaced)
     (property "Reference" "U2" (id 0) (at 124.46 104.14 0)
@@
       (effects (font (size 1.524 1.524)))
     )
-    (property "Footprint" "antmicro-footprints:QFN-56-1EP_8x8mm_P0.5mm_EP5.5.9x5.9mm" (id 2) (at 129.54 162.56 90)
+    (property "Footprint" "arty-mpw-tester-footprints:QFN-56-1EP_8x8mm_P0.5mm_EP5.5.9x5.9mm" (id 2) (at 129.54 162.56 90)
       (effects (font (size 1.524 1.524)) (justify left) hide)
     )
@@
     (pin "2")
   )
-  (symbol (lib_id "antmicroPMICVoltageRegulatorsLinear:TAR5S33UTE85LF") (at 162.56 50.8 0) (unit 1)
+  (symbol (lib_id "arty-mpw-tester:TAR5S33UTE85LF") (at 162.56 50.8 0) (unit 1)
     (in_bom yes) (on_board yes) (fields_autoplaced)
     (property "Reference" "U11" (id 0) (at 162.56 40.64 0))
     (property "Value" "TAR5S33UTE85LF" (id 1) (at 162.56 43.18 0))
-    (property "Footprint" "antmicro-footprints:SOT-353" (id 2) (at 165.1 77.47 0)
+    (property "Footprint" "arty-mpw-tester-footprints:SOT-353" (id 2) (at 165.1 77.47 0)
       (effects (font (size 1.27 1.27)) hide)
     )
@@
     (pin "2")
   )
-  (symbol (lib_id "antmicroFerriteBeadsandChips:BLM18SG121TN1D") (at 190.5 48.26 0) (unit 1)
+  (symbol (lib_id "arty-mpw-tester:BLM18SG121TN1D") (at 190.5 48.26 0) (unit 1)
     (in_bom yes) (on_board yes)
     (property "Reference" "FB3" (id 0) (at 190.5 40.64 0)
@@
       (effects (font (size 1.524 1.524)))
     )
-    (property "Footprint" "antmicro-footprints:0603-res" (id 2) (at 195.58 43.18 0)
+    (property "Footprint" "arty-mpw-tester-footprints:0603-res" (id 2) (at 195.58 43.18 0)
       (effects (font (size 1.524 1.524)) (justify left) hide)
     )
@@
     (pin "4")
   )
-  (symbol (lib_id "antmicroCapacitors0603:C_10u_0603") (at 182.88 59.69 0) (unit 1)
+  (symbol (lib_id "arty-mpw-tester:C_10u_0603") (at 182.88 59.69 0) (unit 1)
     (in_bom yes) (on_board yes) (fields_autoplaced)
     (property "Reference" "C8" (id 0) (at 185.801 58.8554 0)
@@
       (effects (font (size 1.524 1.524)) hide)
     )
-    (property "Footprint" "antmicro-footprints:0603-cap" (id 2) (at 187.96 54.61 0)
+    (property "Footprint" "arty-mpw-tester-footprints:0603-cap" (id 2) (at 187.96 54.61 0)
       (effects (font (size 1.524 1.524)) (justify left) hide)
     )
@@
     (pin "2")
   )
-  (symbol (lib_id "antmicroFerriteBeadsandChips:BLM18SG121TN1D") (at 40.64 259.08 0) (unit 1)
+  (symbol (lib_id "arty-mpw-tester:BLM18SG121TN1D") (at 40.64 259.08 0) (unit 1)
     (in_bom yes) (on_board yes)
     (property "Reference" "FB1" (id 0) (at 40.64 251.46 0)
@@
       (effects (font (size 1.524 1.524)))
     )
-    (property "Footprint" "antmicro-footprints:0603-res" (id 2) (at 45.72 254 0)
+    (property "Footprint" "arty-mpw-tester-footprints:0603-res" (id 2) (at 45.72 254 0)
       (effects (font (size 1.524 1.524)) (justify left) hide)
     )
@@
     (pin "2")
   )
-  (symbol (lib_id "antmicroFerriteBeadsandChips:BLM18SG121TN1D") (at 97.79 259.08 0) (unit 1)
+  (symbol (lib_id "arty-mpw-tester:BLM18SG121TN1D") (at 97.79 259.08 0) (unit 1)
     (in_bom yes) (on_board yes)
     (property "Reference" "FB2" (id 0) (at 97.79 251.46 0)
@@
       (effects (font (size 1.524 1.524)))
     )
-    (property "Footprint" "antmicro-footprints:0603-res" (id 2) (at 102.87 254 0)
-      (effects (font (size 1.524 1.524)) (justify left) hide)
-    )
+    (property "Footprint" "arty-mpw-tester-footprints:0603-res" (id 2) (at 102.87 254 0)
+      (effects (font (size 1.524 1.524)) (justify left) hide)
+    )
