File: arty-mpw-tester.kicad_sch (KiCad schematic)
At the start: 112 parts, among them J1 USB-C_USB4105-GF-A, J14 PinHeader_1x3_P2.54mm_Drill1.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, J15 PinHeader_1x3_P2.54mm_Drill1.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, J18 PinHeader_1x4_P2.54mm_Drill1.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, J19 PinHeader_1x7_P2.54mm_Drill1.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, J2 PinHeader_2x4_P2.54mm_Drill1mm, J20 PinHeader_1x4_P2.54mm_Drill1.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, J3 arty_chipKIT_connector, J4 PinHeader_1x2_P2.54mm_Drill1.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, J5 PinHeader_1x3_P2.54mm_Drill1.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, J6 PinHeader_2x3_P2.54mm_Drill1mm, Q1 DTC014T_SOT-416, SW1 SW_DPDT_JS202011JCQN_SMD, SW2 SW_DPDT_JS202011JCQN_SMD, SW3 SW_DPDT_JS202011JCQN_SMD, U1 SN74LVC1G125_SC70, U10 TPD4E02B04DQA, U2 FT232H_QFN, U3 SN74LVC1G125_SC70, U4 MAX811REUS+T, U5 NTS0102_TSSOP, U6 MCP4661-103E_QFN, U7 Caravel_breakout_flexypin, U8 W25Q32FV_SOIC-8, U9 MIC2211-AAYML, Y1 Oscillator_SMD_12MHz_KX-7, Y2 Oscillator_SMD_10MHz_ECS_2520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

Commit message: [#62395] Perform kmake globlib
Parts:
- C1, C22, C23, C24, C26, C27, C28, C29, C3, C30, C31, C32, C35, C36: footprint arty-mpw-tester-footprints:C_0603_1608Metric -> antmicro-footprints:C_0603_1608Metric; symbol arty-mpw-tester:C_1u_0603 -> antmicroCapacitors0603:C_1u_0603
- C10, C11, C13, C14, C15, C16, C18, C19, C20, C21, C25, C33, C34, C37, C4, C5, C7, C8: footprint arty-mpw-tester-footprints:C_0603_1608Metric -> antmicro-footprints:C_0603_1608Metric; symbol arty-mpw-tester:C_100n_0603 -> antmicroCapacitors0603:C_100n_0603
- C12, C2: footprint arty-mpw-tester-footprints:C_0603_1608Metric -> antmicro-footprints:C_0603_1608Metric; symbol arty-mpw-tester:C_4u7_0603 -> antmicroCapacitors0603:C_4u7_0603
- C17: footprint arty-mpw-tester-footprints:C_0603_1608Metric -> antmicro-footprints:C_0603_1608Metric; symbol arty-mpw-tester:C_10n_0603 -> antmicroCapacitors0603:C_10n_0603
- C6, C9: footprint arty-mpw-tester-footprints:C_0603_1608Metric -> antmicro-footprints:C_0603_1608Metric; symbol arty-mpw-tester:C_18p_0603 -> antmicroCapacitors0603:C_18p_0603
- D1, D2, D3, D4: footprint arty-mpw-tester-footprints:LED_0603_1608Metric_G -> antmicro-footprints:LED_0603_1608Metric_G; symbol arty-mpw-tester:LED_G_0603_KP-1608ZGC -> antmicroLEDIndicationDiscrete:LED_G_0603_KP-1608ZGC
- D5, D6, D9: footprint arty-mpw-tester-footprints:D_SOD-323F -> antmicro-footprints:D_SOD-323F; symbol arty-mpw-tester:PMEG6002EJ,115 -> antmicroDiodesRectifiersSingle:PMEG6002EJ,115
- D7, D8: footprint arty-mpw-tester-footprints:D_SOD-123 -> antmicro-footprints:D_SOD-123; symbol arty-mpw-tester:1N5819HW-7-F -> antmicroDiodesRectifiersSingle:1N5819HW-7-F
- J1: footprint arty-mpw-tester-footprints:USB-C_GCT_USB4105-GF-A -> antmicro-footprints:USB-C_Receptacle_GCT_USB4105-GF-A; symbol arty-mpw-tester:USB-C_USB4105-GF-A -> antmicroUSBConnectors:USB-C_GCT_USB4105-GF-A
- J14, J15, J5: footprint arty-mpw-tester-footprints:PinHeader_1x3_P2.54_Drill1.1mm -> antmicro-footprints:PinHeader_1x3_P2.54mm_Drill1.1mm; symbol arty-mpw-tester:PinHeader_1x3_P2.54mm_Drill1.1mm -> antmicroGenericPinHeaders:PinHeader_1x3_P2.54mm_Drill1.1mm
- J18, J20: footprint arty-mpw-tester-footprints:PinHeader_1x4_P2.54mm_Drill1.02mm -> antmicro-footprints:PinHeader_1x4_P2.54mm_Drill1.1mm; symbol arty-mpw-tester:PinHeader_1x4_P2.54mm_Drill1.1mm -> antmicroGenericPinHeaders:PinHeader_1x4_P2.54mm_Drill1.1mm
- J19: footprint arty-mpw-tester-footprints:PinHeader_1x7_P2.54mm -> antmicro-footprints:PinHeader_1x7_P2.54mm_Drill1.1mm; symbol arty-mpw-tester:PinHeader_1x7_P2.54mm_Drill1.1mm -> antmicroGenericPinHeaders:PinHeader_1x7_P2.54mm_Drill1.1mm
- J3: footprint arty-mpw-tester-footprints:ARTY_A7_SHIELD -> antmicro-footprints:ARTY_A7_SHIELD; symbol arty-mpw-tester:arty_chipKIT_connector -> antmicroModules:arty_chipKIT_connector
- J4: footprint arty-mpw-tester-footprints:PinHeader_1x2_P2.54_Drill0.9mm -> antmicro-footprints:PinHeader_1x2_P2.54_Drill0.9mm; symbol arty-mpw-tester:PinHeader_1x2_P2.54mm_Drill1.1mm -> antmicroGenericPinHeaders:PinHeader_1x2_P2.54mm_Drill1.1mm
- N1: footprint arty-mpw-tester-footprints:antmicro-logo_scaled_12mm -> antmicro-footprints:antmicro-logo; symbol arty-mpw-tester:antmicro_logo -> antmicroMechanicalParts:antmicro_logo
- N2: footprint arty-mpw-tester-footprints:oshw-logo -> antmicro-footprints:oshw-logo; symbol arty-mpw-tester:oshw_logo -> antmicroMechanicalParts:oshw_logo
- Q1: footprint arty-mpw-tester-footprints:SOT-416 -> antmicro-footprints:SOT-416; symbol arty-mpw-tester:DTC014T_SOT-416 -> antmicroTransistorsBipolarSingle:DTC014T_SOT-416
- R1, R16, R17, R18, R19, R20, R21, R26, R28, R30, R32, R33, R34, R6: footprint arty-mpw-tester-footprints:R_0603_1608Metric -> antmicro-footprints:R_0603_1608Metric; symbol arty-mpw-tester:R_10k_0603 -> antmicroResistors0603:R_10k_0603
- R10, R12, R13, R9: footprint arty-mpw-tester-footprints:R_0603_1608Metric -> antmicro-footprints:R_0603_1608Metric; symbol arty-mpw-tester:R_470R_0603 -> antmicroResistors0603:R_470R_0603
- R11, R14, R15, R29, R35, R8: footprint arty-mpw-tester-footprints:R_0603_1608Metric -> antmicro-footprints:R_0603_1608Metric; symbol arty-mpw-tester:R_0R_0603 -> antmicroResistors0603:R_0R_0603
- R2, R3: footprint arty-mpw-tester-footprints:R_0603_1608Metric -> antmicro-footprints:R_0603_1608Metric; symbol arty-mpw-tester:R_5k1_0603 -> antmicroResistors0603:R_5k1_0603
- R22: footprint arty-mpw-tester-footprints:R_0603_1608Metric -> antmicro-footprints:R_0603_1608Metric; symbol arty-mpw-tester:R_68k_0603 -> antmicroResistors0603:R_68k_0603
- R23: footprint arty-mpw-tester-footprints:R_0603_1608Metric -> antmicro-footprints:R_0603_1608Metric; symbol arty-mpw-tester:R_41k2_0603 -> antmicroResistors0603:R_41k2_0603
- R24: footprint arty-mpw-tester-footprints:R_0603_1608Metric -> antmicro-footprints:R_0603_1608Metric; symbol arty-mpw-tester:R_15k_0603 -> antmicroResistors0603:R_15k_0603
- R25: footprint arty-mpw-tester-footprints:R_0603_1608Metric -> antmicro-footprints:R_0603_1608Metric; symbol arty-mpw-tester:R_34k_0603 -> antmicroResistors0603:R_34k_0603
- R27, R31: footprint arty-mpw-tester-footprints:R_0603_1608Metric -> antmicro-footprints:R_0603_1608Metric; symbol arty-mpw-tester:R_4k7_0603 -> antmicroResistors0603:R_4k7_0603
- R4, R5: footprint arty-mpw-tester-footprints:R_0402_1005Metric -> antmicro-footprints:R_0402_1005Metric; symbol arty-mpw-tester:R_0R_0402 -> antmicroResistors0402:R_0R_0402
- R7: footprint arty-mpw-tester-footprints:R_0603_1608Metric -> antmicro-footprints:R_0603_1608Metric; symbol arty-mpw-tester:R_12k_0603 -> antmicroResistors0603:R_12k_0603
- S1: footprint arty-mpw-tester-footprints:SW_SPST_4.2x2.8 -> antmicro-footprints:SW_KMR211NGLFS_SMD; symbol arty-mpw-tester:SW_SPST_KMR211NGLFS -> antmicroPushbuttonSwitches:SW_KMR211NGLFS_SMD
- SW1, SW2, SW3: footprint arty-mpw-tester-footprints:SW_DPDT_CnK_JS202011JCQN_SMD -> antmicro-footprints:SW_DPDT_CnK_JS202011JCQN_SMD; symbol arty-mpw-tester:SW_DPDT_JS202011JCQN_SMD -> antmicroSlideSwitches:SW_DPDT_JS202011JCQN_SMD
- TP1: footprint arty-mpw-tester-footprints:PROBE_PAD_1206 -> antmicro-footprints:TP_1206_SMD_RCW-0C; symbol arty-mpw-tester:TestPoint_Probe_1206_RCW-0C -> antmicroTestPoints:TP_1206_SMD_RCW-0C
- U1, U3: footprint arty-mpw-tester-footprints:SOT-353 -> antmicro-footprints:SOT-353; symbol arty-mpw-tester:SN74LVC1G125_SC70 -> antmicroLogicBuffersDriversReceiversTransceivers:SN74LVC1G125_SC70
- U10: footprint arty-mpw-tester-footprints:USON-10_2.5x1mm_P0.5mm -> antmicro-footprints:USON-10_2.5x1mm_P0.5mm; symbol arty-mpw-tester:TPD4E02B04DQA -> antmicroTVSDiodes:TPD4E02B04DQA
- U2: footprint arty-mpw-tester-footprints:QFN-48-1EP_8x8mm_P0.5mm_EP6.2x6.2mm_FT232HQ_marking -> antmicro-footprints:QFN-48-1EP_8x8mm_P0.5mm_EP6.2x6.2mm_FT232HQ_marking; symbol arty-mpw-tester:FT232H_QFN -> antmicroInterfaceControllers:FT232H_QFN
- U4: footprint arty-mpw-tester-footprints:SOT-143-4 -> antmicro-footprints:SOT-143-4; symbol arty-mpw-tester:MAX811REUS+T -> antmicroPMICPowerSequencers:MAX811REUS+T
- U5: footprint arty-mpw-tester-footprints:TSSOP-8_3x3mm_P0.65mm -> antmicro-footprints:TSSOP-8_3x3mm_P0.65mm; symbol arty-mpw-tester:NTS0102_TSSOP -> antmicroLogicTranslatorsLevelShifters:NTS0102_TSSOP
- U6: footprint arty-mpw-tester-footprints:QFN-16_1EP_4x4mm_P0.65mm -> antmicro-footprints:QFN-16-1EP_4x4mm_P0.65mm; symbol arty-mpw-tester:MCP4661-103E_QFN -> antmicroInterfaceIOExpanders:MCP4661-103E_QFN
- U7: footprint arty-mpw-tester-footprints:Flexypin_56_P1.27mm_Caravel_Breakout -> antmicro-footprints:Flexypin_56_P1.27mm_Caravel_Breakout; symbol arty-mpw-tester:Caravel_breakout_flexypin -> antmicroModules:Caravel_breakout_flexypin
- U8: footprint arty-mpw-tester-footprints:SOIC127P790X216-8N -> antmicro-footprints:SOIC-8_5.3x5.3x2mm_P1.27mm; symbol arty-mpw-tester:W25Q32FV_SOIC-8 -> antmicroMemory:W25Q32FV_SOIC-8
- U9: footprint arty-mpw-tester-footprints:DFN-10-1EP_3x3mm -> antmicro-footprints:DFN-10-1EP_3x3mm; symbol arty-mpw-tester:MIC2211-AAYML -> antmicroPMICVoltageRegulatorsLinear:MIC2211-AAYML
- Y2: footprint arty-mpw-tester-footprints:Oscillator_SMD_ECS_2520MV_2.5x2mm -> antmicro-footprints:Oscillator_SMD_ECS_2520MV_2.5x2mm; symbol arty-mpw-tester:Oscillator_SMD_10MHz_ECS_2520MV -> antmicroOscillators:Oscillator_10MHz_ESC_2520MV

Commit message: [#62395] Update symbols D,J,N,Q,SW,U,Y references
Parts:
- removed J6: PinHeader_2x3_P2.54mm_Drill1mm, arty-mpw-tester-footprints:PinHeader_2x3_P2.54mm_Drill1mm, symbol arty-mpw-tester:PinHeader_2x3_P2.54mm_Drill1mm
- removed Y1: Oscillator_SMD_12MHz_KX-7, arty-mpw-tester-footprints:Oscillator_SMD_Geyer_KX-7-4Pin_3.2x2.5mm, symbol arty-mpw-tester:Oscillator_SMD_12MHz_KX-7
- added J6: PinHeader_2x3_P2.54mm_Drill1.1mm, antmicro-footprints:PinHeader_2x3_P2.54mm_Drill1.1mm, symbol antmicroGenericPinHeaders:PinHeader_2x3_P2.54mm_Drill1.1mm
- added Y1: Resonator_12MHz_ABM8G, antmicro-footprints:Resonator_SMD_Abracon_ABM8G_3.2x2.5mm, symbol antmicroResonators:Resonator_12MHz_ABM8G
- D1, D2, D3, D4: Color (none) -> Green
- J1: value USB-C_USB4105-GF-A -> USB-C_GCT_USB4105-GF-A
- N1, N2: now left out of the parts list
- U2: Manufacturer FTDI -> FTDI Chip
- U4: Manufacturer Maxim Integrated -> Maxim Integrated Products
- U6, U9: Manufacturer Microchip -> Microchip Technology
- U7: MPN caravel_breakout -> Flexypin; now left out of the parts list
- Y2: value Oscillator_SMD_10MHz_ECS_2520MV -> Oscillator_10MHz_ESC_2520MV; Manufacturer ECS Inc. -> ECS Inc. International; VAL 10 MHz -> (none); Val (none) -> 10 MHz
Connections:
- net +1V8: now also J6.2, J6.4, J6.6
- net +3V3: now also D3.2 (A), D4.2 (A); no longer D3.1, D4.1
- net 5V0: now also D7.1 (C), D8.1 (C); no longer D7.K, D8.K
- net 5V0_ARTY: now also D8.2 (A); no longer D8.A
- net ARTY_~{MR}: now also D9.1 (C); no longer D9.K
- net FTDI_3V3: now also D1.2 (A), D2.2 (A); no longer D1.1, D2.1
- net FTDI_~{MR}: now also D6.1 (C); no longer D6.K
- net FTDI_~{UART_EN}: now also D5.1 (C); no longer D5.K
- net GND: now also Y1.2 (SH), Y1.4 (SH)
- net USB_DN: no longer J1.B7 (D-)
- net USB_DP: now also J1.B7 (D_{B}-)
- net VBUS: now also D7.2 (A); no longer D7.A
- net VCCD: now also J6.1
- net VCCD1: now also J6.3
- net VCCD2: now also J6.5
- net XIN: now also Y1.1
- net XOUT: now also Y1.3
- net ~{MR}: now also D6.2 (A), D9.2 (A); no longer D6.A, D9.A
- net ~{UART_EN}: now also D5.2 (A); no longer D5.A
- net at R12.2: now also D3.1 (C); no longer D3.2
- net at R9.2: now also D1.1 (C); no longer D1.2
- net at R10.2: now also D2.1 (C); no longer D2.2
- net at R13.2: now also D4.1 (C); no longer D4.2
Other:
- moved on the sheet: C1, C10, C12, C13, C15, C16, C17, C19, C20, C21, C22, C24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

Commit message: [#62395] Update R,C and allign schematic
Parts:
- C1, C22, C23, C24, C26, C27, C28, C29, C3, C30, C31, C32, C35, C36: Manufacturer Walsin -> KYOCERA AVX
- R26, R27, R31: DNP DNP -> (none); now in the parts list
- S1: value SW_SPST_KMR211NGLFS -> SW_KMR211NGLFS_SMD
- TP1: value TestPoint_Probe_1206_RCW-0C -> TP_1206_SMD_RCW-0C
Connections:
- net GND: now also S1.3; no longer S1.2
- net USB_DN: now also J1.B7 (D_{B}-)
- net USB_DP: no longer J1.B7 (D_{B}-)
- net ~{MR}: now also S1.2; no longer S1.3
Other:
- moved on the sheet: C11, C14, C2, C22, C23, C24, C26, C28, C29, C31, C32, C33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

Commit message: [#62395] Update J2
Parts:
- removed J2: PinHeader_2x4_P2.54mm_Drill1mm, arty-mpw-tester-footprints:PinHeader_2x4_P2.54mm_Drill1mm, symbol arty-mpw-tester:PinHeader_2x4_P2.54mm_Drill1mm
- added J2: PinHeader_2x4_P2.54mm_Drill1.02mm, antmicro-footprints:PinHeader_2x4_P2.54mm_Drill1.02mm, symbol antmicroGenericPinHeaders:PinHeader_2x4_P2.54mm_Drill1.02mm
Connections:
- net +3V3: now also J2.2, J2.4, J2.6, J2.8
- net VDDA: now also J2.7
- net VDDA1: now also J2.5
- net VDDA2: now also J2.3
- net VDDIO: now also J2.1
Other:
- moved on the sheet: C12, C13, C15, C16, C22, C23, C24, C26, C27, C28, C29, C30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

Commit message: [#62395] Update J, N footprints
Parts:
- N1: footprint antmicro-footprints:antmicro-logo -> antmicro-footprints:antmicro-logo_scaled_12mm
Changed lines of the file:
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@@
       (effects (font (size 1.27 1.27) (thickness 0.15)) (justify left))
     )
-    (property "Footprint" "antmicro-footprints:antmicro-logo" (at 320.04 250.825 0)
+    (property "Footprint" "antmicro-footprints:antmicro-logo_scaled_12mm" (at 320.04 250.825 0)
       (effects (font (size 1.27 1.27) (thickness 0.15)) (justify left bottom) hide)
     )
